File: hardware/logicboard/ledpanel-001.sch (EAGLE design)
At the start: 7 parts

Commit message: Changed dimension.
Parts:
- removed GREENA, REDA: (no value), SparkFun-Connectors:CONN_04JST-PTH
- added GRN, RED: (no value), SparkFun-Connectors:CONN_04JST-PTH-VERT
- PWR: device SparkFun-Connectors:CONN_02JST-PTH-2 -> SparkFun-Connectors:CONN_02-JST-2-PTH-NO_SILK
Connections:
- net GREEN1: now also GRN.1; no longer GREENA.1
- net GREEN2: now also GRN.2; no longer GREENA.2
- net GREEN3: now also GRN.3; no longer GREENA.3
- net GREEN4: now also GRN.4; no longer GREENA.4
- net RED1: now also RED.1; no longer REDA.1
- net RED2: now also RED.2; no longer REDA.2
- net RED3: now also RED.3; no longer REDA.3
- net RED4: now also RED.4; no longer REDA.4
Changed lines of the file:
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@@
 <?xml version="1.0" encoding="utf-8"?>
 <!DOCTYPE eagle SYSTEM "eagle.dtd">
-<eagle version="8.6.3">
+<eagle version="8.7.0">
 <drawing>
 <settings>
@@
 <setting verticaltext="up"/>
 </settings>
-<grid distance="0.1" unitdist="inch" unit="inch" style="lines" multiple="1" display="yes" altdistance="0.01" altunitdist="inch" altunit="inch"/>
+<grid distance="0.1" unitdist="inch" unit="inch" style="lines" multiple="1" display="no" altdistance="0.01" altunitdist="inch" altunit="inch"/>
 <layers>
 <layer number="1" name="Top" color="4" fill="1" visible="no" active="no"/>
@@
 </classes>
 <parts>
-<part name="PWR" library="SparkFun-Connectors" deviceset="CONN_02" device="JST-PTH-2"/>
+<part name="PWR" library="SparkFun-Connectors" deviceset="CONN_02" device="-JST-2-PTH-NO_SILK"/>
 <part name="SUPPLY1" library="supply2" library_urn="urn:adsk.eagle:library:372" deviceset="GND" device=""/>
 <part name="LD4" library="led" library_urn="urn:adsk.eagle:library:259" deviceset="DUOLED-RG-C" device="" package3d_urn="urn:adsk.eagle:package:15851/1"/>
@@
 <part name="LD2" library="led" library_urn="urn:adsk.eagle:library:259" deviceset="DUOLED-RG-C" device="" package3d_urn="urn:adsk.eagle:package:15851/1"/>
 <part name="LD1" library="led" library_urn="urn:adsk.eagle:library:259" deviceset="DUOLED-RG-C" device="" package3d_urn="urn:adsk.eagle:package:15851/1"/>
-<part name="REDA" library="SparkFun-Connectors" deviceset="CONN_04" device="JST-PTH"/>
-<part name="GREENA" library="SparkFun-Connectors" deviceset="CONN_04" device="JST-PTH"/>
+<part name="RED" library="SparkFun-Connectors" deviceset="CONN_04" device="JST-PTH-VERT"/>
+<part name="GRN" library="SparkFun-Connectors" deviceset="CONN_04" device="JST-PTH-VERT"/>
 </parts>
 <sheets>
@@
 <instance part="LD2" gate="G$1" x="58.42" y="38.1" rot="R90"/>
 <instance part="LD1" gate="G$1" x="58.42" y="48.26" rot="R90"/>
-<instance part="REDA" gate="G$1" x="10.16" y="27.94"/>
-<instance part="GREENA" gate="G$1" x="10.16" y="43.18"/>
+<instance part="RED" gate="G$1" x="10.16" y="27.94"/>
+<instance part="GRN" gate="G$1" x="10.16" y="43.18"/>
 </instances>
 <busses>
@@
 </segment>
 <segment>
-<pinref part="GREENA" gate="G$1" pin="1"/>
+<pinref part="GRN" gate="G$1" pin="1"/>
 <wire x1="15.24" y1="40.64" x2="17.78" y2="43.18" width="0.1524" layer="91" curve="90"/>
 </segment>
@@
 </segment>
 <segment>
-<pinref part="GREENA" gate="G$1" pin="2"/>
+<pinref part="GRN" gate="G$1" pin="2"/>
 <wire x1="15.24" y1="43.18" x2="17.78" y2="45.72" width="0.1524" layer="91" curve="90"/>
 </segment>
@@
 </segment>
 <segment>
-<pinref part="GREENA" gate="G$1" pin="3"/>
+<pinref part="GRN" gate="G$1" pin="3"/>
 <wire x1="15.24" y1="45.72" x2="17.78" y2="48.26" width="0.1524" layer="91" curve="90"/>
 </segment>
@@
 </segment>
 <segment>
-<pinref part="GREENA" gate="G$1" pin="4"/>
+<pinref part="GRN" gate="G$1" pin="4"/>
 <wire x1="15.24" y1="48.26" x2="17.78" y2="50.8" width="0.1524" layer="91" curve="90"/>
 </segment>
@@
 </segment>
 <segment>
-<pinref part="REDA" gate="G$1" pin="4"/>
+<pinref part="RED" gate="G$1" pin="4"/>
 <wire x1="15.24" y1="33.02" x2="17.78" y2="30.48" width="0.1524" layer="91" curve="-90"/>
 </segment>
@@
 </segment>
 <segment>
-<pinref part="REDA" gate="G$1" pin="3"/>
+<pinref part="RED" gate="G$1" pin="3"/>
 <wire x1="15.24" y1="30.48" x2="17.78" y2="27.94" width="0.1524" layer="91" curve="-90"/>
 </segment>
@@
 </segment>
 <segment>
-<pinref part="REDA" gate="G$1" pin="2"/>
+<pinref part="RED" gate="G$1" pin="2"/>
 <wire x1="15.24" y1="27.94" x2="17.78" y2="25.4" width="0.1524" layer="91" curve="-90"/>
 </segment>
@@
 </segment>
 <segment>
-<pinref part="REDA" gate="G$1" pin="1"/>
+<pinref part="RED" gate="G$1" pin="1"/>
 <wire x1="15.24" y1="25.4" x2="17.78" y2="22.86" width="0.1524" layer="91" curve="-90"/>
 </segment>
@@
 </sheet>
 </sheets>
+<errors>
+</errors>
 </schematic>
 </drawing>
